File: Septh_left/Septh_left.kicad_pcb (KiCad board)
At the start: 2 copper layers, 173.1 x 127.5 mm, 87 parts, among them J1 MJ-4PP-9, P1 i2C, P2 i2C, SW00 SW_Push, SW1 SW_PUSH, SW10 SW_PUSH, SW11 SW_PUSH, SW12 SW_PUSH, SW13 SW_PUSH, SW14 SW_PUSH, SW15 SW_PUSH, SW16 SW_PUSH, SW17 SW_PUSH, SW18 SW_PUSH, SW19 SW_PUSH, SW2 SW_PUSH, SW20 SW_PUSH, SW21 SW_PUSH, SW22 SW_PUSH, SW23 SW_PUSH, SW24 SW_PUSH, SW25 SW_PUSH, SW26 SW_PUSH, SW27 SW_PUSH, SW28 SW_PUSH, SW29 SW_PUSH, SW3 SW_PUSH, SW30 SW_PUSH, SW31 SW_PUSH, SW32 RotaryEncoder_Switch, SW33 SW_PUSH, SW34 SW_PUSH, SW35 SW_PUSH, SW4 SW_PUSH, SW5 SW_PUSH, SW6 SW_PUSH, SW7 SW_PUSH, SW8 SW_PUSH, SW9 SW_PUSH, U1 ProMicro

Commit message: Add files via upload
Parts:
- removed the Ref** at (-114.5, 31.0)
- added Ref**: Val**, kbd_Hole:m2_Screw_Hole, F.Cu at (152.5, 84.5)
- added Ref**: Val**, kbd_Hole:m2_Screw_Hole, F.Cu at (153.0, 48.0)
- added Ref**: Val**, kbd_Hole:m2_Screw_Hole, F.Cu at (118.5, 140.0)
- J1: moved to F.Cu
- SW32: value RotaryEncoder_Switch -> SW_PUSH; footprint kbd_Parts:RotaryEncoder_EC12E -> my-foot:Choc_v2_Hotswap_1u_Narrow; moved to B.Cu
- SW35: value SW_PUSH -> RotaryEncoder_Switch; footprint my-foot:Choc_v2_予備配線 -> kbd_Parts:RotaryEncoder_EC12E
- moved Ref** 263.1 mm to (151.5, 115.5)
- moved Ref** 219.5 mm to (172.0, 152.0)
- moved SW00 207.0 mm to (84.5, 35.0)
- moved Ref** 151.6 mm to (78.0, 56.5)
- moved Ref** 137.3 mm to (90.0, 111.0)
- moved D34 97.5 mm to (159.0, 91.5)
- moved D33 95.9 mm to (159.0, 87.0)
- moved SW35 87.9 mm to (165.0, 108.0), turned to 180 degrees
- moved SW34 87.0 mm to (168.0, 94.0), turned to 180 degrees
- moved D35 86.5 mm to (165.0, 119.0)
- moved SW33 84.7 mm to (168.0, 89.0), turned to 180 degrees
- moved D41 73.8 mm to (110.0, 112.0)
- moved D42 72.7 mm to (132.0, 113.5)
- moved D30 64.9 mm to (162.0, 146.5)
- moved D20 56.8 mm to (136.5, 133.5)
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Connections:
- U1 pad 17: col0 -> col3
- U1 pad 18: col1 -> col2
- U1 pad 19: col2 -> col1
- U1 pad 20: col3 -> col0
Routing:
- net row3: track 0.00 -> 224.8 mm, vias 0 -> 9
- net row4: track 0.00 -> 223.5 mm, vias 0 -> 3
- net GND: track 0.00 -> 219.5 mm, vias 0 -> 5
- net col2: track 0.00 -> 197.1 mm, vias 0 -> 6
- net row2: track 0.00 -> 189.7 mm, vias 0 -> 7
- net col0: track 0.00 -> 187.8 mm, vias 0 -> 3
- net col1: track 0.00 -> 183.5 mm, vias 0 -> 10
- net roB: track 0.00 -> 178.7 mm, vias 0 -> 2
- net col3: track 0.00 -> 178.5 mm, vias 0 -> 8
- net row1: track 0.00 -> 175.2 mm, vias 0 -> 7
- net roA: track 0.00 -> 172.8 mm, vias 0 -> 2
- net row0: track 0.00 -> 166.8 mm, vias 0 -> 9
- net Net-(D41-A): track 0.00 -> 140.7 mm, vias 0 -> 7
- net Net-(D42-A): track 0.00 -> 126.8 mm, vias 0 -> 7
- net Net-(D43-A): track 0.00 -> 104.3 mm, vias 0 -> 7
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Other:
- board size 173.1 x 127.5 mm -> 356 x 128.5 mm
- board text added: "Septh_right Ver1.0"
- board text removed: "MicElgo_right_Ver1.0"
