File: Septh_left/Septh_left.kicad_sch (KiCad schematic)
At the start: 80 parts, among them J1 MJ-4PP-9, P1 i2C, P2 i2C, SW00 SW_Push, SW1 SW_PUSH, SW10 SW_PUSH, SW11 SW_PUSH, SW12 SW_PUSH, SW13 SW_PUSH, SW14 SW_PUSH, SW15 SW_PUSH, SW16 SW_PUSH, SW17 SW_PUSH, SW18 SW_PUSH, SW19 SW_PUSH, SW2 SW_PUSH, SW20 SW_PUSH, SW21 SW_PUSH, SW22 SW_PUSH, SW23 SW_PUSH, SW24 SW_PUSH, SW25 SW_PUSH, SW26 SW_PUSH, SW27 SW_PUSH, SW28 SW_PUSH, SW29 SW_PUSH, SW3 SW_PUSH, SW30 SW_PUSH, SW31 SW_PUSH, SW32 RotaryEncoder_Switch, SW33 SW_PUSH, SW34 SW_PUSH, SW35 SW_PUSH, SW4 SW_PUSH, SW5 SW_PUSH, SW6 SW_PUSH, SW7 SW_PUSH, SW8 SW_PUSH, SW9 SW_PUSH, U1 ProMicro

Commit message: Add files via upload
Parts:
- SW32: renamed from SW33; footprint my-foot:Choc_v2_予備配線 -> my-foot:Choc_v2_Hotswap_1u_Narrow
- renumbered SW35 to SW33, SW32 to SW35
Connections:
- net col0: now also U1.20 (F4/A3); no longer U1.17 (F7/A0)
- net col1: now also U1.19 (F5/A2); no longer U1.18 (F6/A1)
- net col2: now also U1.18 (F6/A1); no longer U1.19 (F5/A2)
- net col3: now also U1.17 (F7/A0); no longer U1.20 (F4/A3)
- net at D33.1 (K): now also SW33.2; no longer SW32.2
- net at D32.1 (K): now also SW32.2; no longer SW35.S1
- net at D35.1 (K): now also SW35.S1; no longer SW33.2
- no-connect marks 3 -> 4
Other:
- moved on the sheet: SW32, SW33, SW35
